File: RPi_Hat.kicad_pcb (KiCad board)
At the start: 2 copper layers, 65 x 56.5 mm, 18 parts, among them J1 RPi_GPIO, P1 CONN_01X02, U1 MCP1754ST-3302E/MB, U2 74LS125, U3 AWA24S, U4 AWA24S, U5 DS3231

Commit message: cleanup of old files, First production version
Connections:
- U1 pad 4: (no net) -> GND
Routing:
- net GND: track 27.4 -> 33.9 mm, vias 12 -> 14
- net (no net): track 0.76 -> 0.00 mm
Other:
- board text added: "B52/CHANNEL/Z REV1/2016/11 E/OVERTON"
- board text removed: "Bot Radio v0 E. Overton, 11/2016"
- board text removed: "Camera Flex Slot (Optional)"
- board text removed: "Dimensions taken from https://github.com/raspberrypi/hats/blob/master/hat-board-mechanical.pdf"
- board text removed: "Select one of these board edges depending upon the type of socket that is used."
